File: pcb/eagle/inkubator.brd (EAGLE design)
At the start: 71.1 x 50.5 mm, 34 parts, among them Q1 BT138-600, Q2 BT138-600, U1 L78L33ABUTR, U2 MOC3063, U3 MOC3063

Commit message: Первая версия печатной платы
Parts:
- moved R2 20.2 mm to (57.0, 10.5), turned to 90 degrees
- moved R3 20.0 mm to (56.1, 22.2), turned to 270 degrees
- moved U$3 10.9 mm to (52.1, 8.89), turned to 90 degrees
- moved U$2 8.98 mm to (52.1, 12.7), turned to 270 degrees
- moved 1WIRE 5.24 mm to (47.0, 11.4), turned to 270 degrees
- moved JP2 1.27 mm to (59.7, 27.9)
- moved R12 1.25 mm to (49.9, 16.6)
Routing:
- net 1W: track 11.3 -> 31.5 mm
- net +3V3: track 29.6 -> 43.9 mm
- net N$1: track 0.00 -> 8.90 mm
- net GND: track 22.1 -> 30.9 mm
- net N$14: track 0.00 -> 2.58 mm
- net 1WTX: track 6.56 -> 7.99 mm
- net SWCLK: track 3.75 -> 5.02 mm
- net SWDIO: track 4.04 -> 5.31 mm
- net NRST: track 18.2 -> 19.2 mm
